Commit message: adjusted urdfs

File: ros2_astra_camera/launch/urdf/astra_pro.urdf (robot description, URDF)
Before this commit: robot astra, 5 links, 4 joints
Joints:
- joint camera_depth_joint: origin xyz=0 -0.02 0 rpy=0 0 0 -> xyz=0 0.0375 0.015 rpy=0 0 0
- joint camera_depth_optical_joint: origin xyz=0 0 0 rpy=1.570896 3.1415926 1.570896 -> xyz=0 0 0 rpy=${pi/2} ${pi} ${pi/2}
- joint camera_rgb_joint: origin xyz=0 -0.045 0 rpy=0 0 0 -> xyz=0 0.0125 0.0150 rpy=0 0 0
- joint camera_rgb_optical_joint: origin xyz=0 0 0 rpy=1.570896 3.1415926 1.570896 -> xyz=0 0 0 rpy=${pi/2} ${pi} ${pi/2}

File: ros2_astra_camera/launch/urdf/astra_pro.urdf.xacro (robot description, xacro)
@@ -1,5 +1,5 @@
 <?xml version="1.0"?>
 <robot xmlns:xacro="http://ros.org/wiki/xacro">
-<robot name="astra">
+<robot name="astra_pro">
   <link name="camera_link"/>
   <link name="camera_rgb_frame"/>
@@ -10,20 +10,20 @@
     <parent link="camera_link"/>
     <child link="camera_rgb_frame"/>
-    <origin xyz="0 -0.045 0" rpy="0 0 0"/>
+    <origin xyz="0 0.0125 0.0150" rpy="0 0 0"/>
   </joint>
   <joint name="camera_depth_joint" type="fixed">
     <parent link="camera_link"/>
     <child link="camera_depth_frame"/>
-    <origin xyz="0 -0.02 0" rpy="0 0 0"/>
+    <origin xyz="0 0.0375 0.015" rpy="0 0 0"/>
   </joint>
   <joint name="camera_rgb_optical_joint" type="fixed">
     <parent link="camera_rgb_frame"/>
     <child link="camera_rgb_optical_frame"/>
-    <origin xyz="0 0 0" rpy="1.570896 3.1415926 1.570896"/>
+    <origin xyz="0 0 0" rpy="${pi/2} ${pi} ${pi/2}"/>
   </joint>
   <joint name="camera_depth_optical_joint" type="fixed">
     <parent link="camera_depth_frame"/>
     <child link="camera_depth_optical_frame"/>
-    <origin xyz="0 0 0" rpy="1.570896 3.1415926 1.570896"/>
+    <origin xyz="0 0 0" rpy="${pi/2} ${pi} ${pi/2}"/>
   </joint>
 </robot>

Commit message: changed urdf structure

File: ros2_astra_camera/launch/urdf/astra_pro.urdf (robot description, URDF)
Before this commit: robot astra, 5 links, 4 joints
Links:
- removed link camera_depth_frame
- removed link camera_depth_optical_frame
- removed link camera_link
- removed link camera_rgb_frame
- removed link camera_rgb_optical_frame
Joints:
- removed joint camera_depth_joint
- removed joint camera_depth_optical_joint
- removed joint camera_rgb_joint
- removed joint camera_rgb_optical_joint

File: ros2_astra_camera/launch/urdf/astra_pro.urdf.xacro (robot description, xacro)
@@ -1,5 +1,4 @@
 <?xml version="1.0"?>
 <robot xmlns:xacro="http://ros.org/wiki/xacro">
-<robot name="astra_pro">
   <link name="camera_link"/>
   <link name="camera_rgb_frame"/>
